Commit message: first test

File: kr_50_r2500_gazebo/urdf/kr_50_r2500_gripper.xacro (robot description, xacro)
@@ -2,5 +2,14 @@
 <robot xmlns:xacro="http://www.ros.org/wiki/xacro">
   <xacro:include filename="$(find kr_50_r2500_gazebo)/urdf/kr_50_r2500_base.xacro" />
-  <xacro:include filename="$(find personal_gripper)/urdf/personal_gripper.xacro" />
+  <!-- <xacro:include filename="$(find personal_gripper)/urdf/personal_gripper.xacro" /> -->
+  <!-- <joint name="gripper_fixed" type="fixed">
+      <origin
+        xyz="0.07 0 0"
+        rpy="0 1.57079632679 0" />
+      <parent link="link6"/>
+      <child link="gripper_base_link"/>
+  </joint> -->
+  <xacro:include filename="$(find parallel_2f_gripper)/urdf/gripper.xacro" />
+  <xacro:gripper prefix=""/>
   <joint name="gripper_fixed" type="fixed">
       <origin
@@ -8,5 +17,5 @@
         rpy="0 1.57079632679 0" />
       <parent link="link6"/>
-      <child link="gripper_base_link"/>
+      <child link="gripper_base"/>
   </joint>
   <!-- <xacro:include filename="$(find kr_50_r2500_gazebo)/urdf/robotiq_arg2f_85_model.xacro" />

Commit message: branched master

File: kr_50_r2500_gazebo/urdf/kr_50_r2500_gripper.xacro (robot description, xacro)
@@ -19,4 +19,24 @@
       <child link="gripper_base"/>
   </joint>
+  <xacro:property name="floor_size_x" value="6" />
+  <xacro:property name="floor_size_y" value="6" />
+  <xacro:property name="floor_size_z" value="0.5" />
+  <xacro:property name="floor" value="0.4 0.4 0.5 1" />
+  <joint name="world_to_floor" type="fixed">
+    <parent link="world"/>
+    <child link="floor"/>
+    <origin xyz="0 0 0"/>
+  </joint>
+  <link name="floor">
+     <collision>
+       <origin xyz="0 0 ${-0.5001*floor_size_z}" rpy="0 0 0" />
+       <geometry>
+         <box size="${floor_size_x} ${floor_size_y} ${floor_size_z}" />
+       </geometry>
+       <material name="White">
+         <color rgba="1 1 1 0.1"/>
+       </material>
+     </collision>
+  </link>
   <!-- <xacro:include filename="$(find kr_50_r2500_gazebo)/urdf/robotiq_arg2f_85_model.xacro" />
   <joint name="gripper_fixed" type="fixed">
