Commit message: robot_name and prefix parametrization added

File: kr_50_r2500_description/urdf/kr_50_r2500_pybullet.xacro (robot description, xacro)
@@ -1,6 +1,11 @@
 <?xml version="1.0"?>
-<robot name="kr_50_r2500" xmlns:xacro="http://www.ros.org/wiki/xacro">
-<xacro:include filename="$(find kr_50_r2500_description)/urdf/kr_50_r2500.xacro" />
-<xacro:property name="prefix" value="''" />
-<xacro:kr_50_r2500 prefix="${prefix}"/>
+<!-- It is required to pass the args: robot_name-->
+<robot name="$(arg robot_name)" xmlns:xacro="http://www.ros.org/wiki/xacro">
+  <xacro:include filename="$(find kr_50_r2500_description)/urdf/kr_50_r2500.xacro" />
+  <xacro:arg name="prefix" default="null"/>
+  <xacro:property name="prefix" value="'$(arg prefix)'" />
+  <xacro:if value="${prefix == 'null'}">
+    <xacro:property name="prefix" value="''" />
+  </xacro:if>
+  <xacro:kr_50_r2500 prefix="${prefix}"/>
 </robot>

File: kr_50_r2500_description/urdf/kr_50_r2500_rviz.xacro (robot description, xacro)
@@ -1,6 +1,11 @@
 <?xml version="1.0"?>
-<robot name="kr_50_r2500" xmlns:xacro="http://www.ros.org/wiki/xacro">
+<!-- It is required to pass the args: robot_name-->
+<robot name="$(arg robot_name)" xmlns:xacro="http://www.ros.org/wiki/xacro">
   <xacro:include filename="$(find kr_50_r2500_description)/urdf/kr_50_r2500.xacro" />
-  <xacro:property name="prefix" value="''" />
+  <xacro:arg name="prefix" default="null"/>
+  <xacro:property name="prefix" value="'$(arg prefix)'" />
+  <xacro:if value="${prefix == 'null'}">
+    <xacro:property name="prefix" value="''" />
+  </xacro:if>
   <xacro:kr_50_r2500 prefix="${prefix}"/>
   <link name="world"/>
