Commit message: moveit config

File: kr_50_r2500_description/urdf/kr_50_r2500.xacro (robot description, xacro)
@@ -20,12 +20,11 @@
   <xacro:property name="joint5_vel_limit" value="3.92699" />    <!--  250°/s -->
   <xacro:property name="joint6_vel_limit" value="5.65487" />    <!--  360°/s -->
-  <xacro:property name="joint1_eff_limit" value="10000" />
-  <xacro:property name="joint2_eff_limit" value="10000" />
-  <xacro:property name="joint3_eff_limit" value="10000" />
-  <xacro:property name="joint4_eff_limit" value="10000" />
-  <xacro:property name="joint5_eff_limit" value="10000" />
-  <xacro:property name="joint6_eff_limit" value="10000" />
-  <link
-    name="${prefix}base_link">
+  <xacro:property name="joint1_eff_limit" value="1000" />
+  <xacro:property name="joint2_eff_limit" value="1000" />
+  <xacro:property name="joint3_eff_limit" value="500" />
+  <xacro:property name="joint4_eff_limit" value="200" />
+  <xacro:property name="joint5_eff_limit" value="200" />
+  <xacro:property name="joint6_eff_limit" value="200" />
+  <link name="${prefix}base_link">
     <inertial>
       <origin
@@ -66,6 +65,5 @@
     </collision>
   </link>
-  <link
-    name="${prefix}link1">
+  <link name="${prefix}link1">
     <inertial>
       <origin
@@ -106,6 +104,5 @@
     </collision>
   </link>
-  <joint
-    name="${prefix}joint1"
+  <joint name="${prefix}joint1"
     type="revolute">
     <origin
@@ -120,6 +117,5 @@
     <limit lower="${joint1_pos_lower_limit}" upper="${joint1_pos_upper_limit}" effort="${joint1_eff_limit}" velocity="${joint1_vel_limit}"/>
   </joint>
-  <link
-    name="${prefix}link2">
+  <link name="${prefix}link2">
     <inertial>
       <origin
@@ -160,6 +156,5 @@
     </collision>
   </link>
-  <joint
-    name="${prefix}joint2"
+  <joint name="${prefix}joint2"
     type="revolute">
     <origin
@@ -174,6 +169,5 @@
     <limit lower="${joint2_pos_lower_limit}" upper="${joint2_pos_upper_limit}" effort="${joint2_eff_limit}" velocity="${joint2_vel_limit}"/>
   </joint>
-  <link
-    name="${prefix}link3">
+  <link name="${prefix}link3">
     <inertial>
       <origin
@@ -214,6 +208,5 @@
     </collision>
   </link>
-  <joint
-    name="${prefix}joint3"
+  <joint name="${prefix}joint3"
     type="revolute">
     <origin
@@ -228,6 +221,5 @@
     <limit lower="${joint3_pos_lower_limit}" upper="${joint3_pos_upper_limit}" effort="${joint3_eff_limit}" velocity="${joint3_vel_limit}"/>
   </joint>
-  <link
-    name="${prefix}link4">
+  <link name="${prefix}link4">
     <inertial>
       <origin
@@ -268,6 +260,5 @@
     </collision>
   </link>
-  <joint
-    name="${prefix}joint4"
+  <joint name="${prefix}joint4"
     type="revolute">
     <origin
@@ -282,6 +273,5 @@
     <limit lower="${joint4_pos_lower_limit}" upper="${joint4_pos_upper_limit}" effort="${joint4_eff_limit}" velocity="${joint4_vel_limit}"/>
   </joint>
-  <link
-    name="${prefix}link5">
+  <link name="${prefix}link5">
     <inertial>
       <origin
@@ -322,6 +312,5 @@
     </collision>
   </link>
-  <joint
-    name="${prefix}joint5"
+  <joint name="${prefix}joint5"
     type="revolute">
     <origin
@@ -336,6 +325,5 @@
     <limit lower="${joint5_pos_lower_limit}" upper="${joint5_pos_upper_limit}" effort="${joint5_eff_limit}" velocity="${joint5_vel_limit}"/>
   </joint>
-  <link
-    name="${prefix}link6">
+  <link name="${prefix}link6">
     <inertial>
       <origin
@@ -376,6 +364,5 @@
     </collision>
   </link>
-  <joint
-    name="${prefix}joint6"
+  <joint name="${prefix}joint6"
     type="revolute">
     <origin
@@ -399,9 +386,6 @@
   <link name="${prefix}flange">
     <inertial>
-      <origin
-        xyz="0 0 0"
-        rpy="0 0 0" />
-      <mass
-        value="0.01" />
+      <origin xyz="0 0 0" rpy="0 0 0" />
+      <mass value="0.01" />
       <inertia
         ixx="0.00001"

File: kr_50_r2500_description/urdf/kr_50_r2500_gazebo.xacro (robot description, xacro)
@@ -11,5 +11,5 @@
     </plugin>
   </gazebo>
-  <gazebo reference="${prefix}flange">
+  <gazebo reference="${prefix}link6_to_flange">
       <provideFeedback>true</provideFeedback>
       <disableFixedJointLumping>true</disableFixedJointLumping>
@@ -18,7 +18,7 @@
   <gazebo>
       <plugin name="ft_sensor" filename="libgazebo_ros_ft_sensor.so">
-          <updateRate>100.0</updateRate>
+          <updateRate>1000.0</updateRate>
           <topicName>${prefix}gripper/wrench</topicName>
-          <jointName>${prefix}flange</jointName>
+          <jointName>${prefix}link6_to_flange</jointName>
       </plugin>
   </gazebo>

Commit message: cleaning up mess

File: kr_50_r2500_description/urdf/kr_50_r2500.xacro (robot description, xacro)
@@ -20,10 +20,10 @@
   <xacro:property name="joint5_vel_limit" value="3.92699" />    <!--  250°/s -->
   <xacro:property name="joint6_vel_limit" value="5.65487" />    <!--  360°/s -->
-  <xacro:property name="joint1_eff_limit" value="1000" />
-  <xacro:property name="joint2_eff_limit" value="1000" />
-  <xacro:property name="joint3_eff_limit" value="500" />
-  <xacro:property name="joint4_eff_limit" value="200" />
-  <xacro:property name="joint5_eff_limit" value="200" />
-  <xacro:property name="joint6_eff_limit" value="200" />
+  <xacro:property name="joint1_eff_limit" value="10000" />
+  <xacro:property name="joint2_eff_limit" value="10000" />
+  <xacro:property name="joint3_eff_limit" value="10000" />
+  <xacro:property name="joint4_eff_limit" value="10000" />
+  <xacro:property name="joint5_eff_limit" value="10000" />
+  <xacro:property name="joint6_eff_limit" value="10000" />
   <link name="${prefix}base_link">
     <inertial>

File: kr_50_r2500_description/urdf/kr_50_r2500_transmission.xacro (robot description, xacro)
@@ -8,5 +8,4 @@
     </joint>
     <actuator name="${prefix}motor1">
-      <hardwareInterface>${interface}</hardwareInterface>
       <mechanicalReduction>1</mechanicalReduction>
     </actuator>
@@ -18,5 +17,4 @@
     </joint>
     <actuator name="${prefix}motor2">
-      <hardwareInterface>${interface}</hardwareInterface>
       <mechanicalReduction>1</mechanicalReduction>
     </actuator>
@@ -28,5 +26,4 @@
     </joint>
     <actuator name="${prefix}motor3">
-      <hardwareInterface>${interface}</hardwareInterface>
       <mechanicalReduction>1</mechanicalReduction>
     </actuator>
@@ -38,5 +35,4 @@
     </joint>
     <actuator name="${prefix}motor4">
-      <hardwareInterface>${interface}</hardwareInterface>
       <mechanicalReduction>1</mechanicalReduction>
     </actuator>
@@ -48,5 +44,4 @@
     </joint>
     <actuator name="${prefix}motor5">
-      <hardwareInterface>${interface}</hardwareInterface>
       <mechanicalReduction>1</mechanicalReduction>
     </actuator>
@@ -58,5 +53,4 @@
     </joint>
     <actuator name="${prefix}motor6">
-      <hardwareInterface>${interface}</hardwareInterface>
       <mechanicalReduction>1</mechanicalReduction>
     </actuator>

Commit message: added pybullet

File: kr_50_r2500_description/urdf/kr_50_r2500.xacro (robot description, xacro)
@@ -1,23 +1,23 @@
 <?xml version="1.0"?>
 <robot  xmlns:xacro="http://www.ros.org/wiki/xacro">
-  <xacro:macro name="kr_50_r2500"  params="prefix:='' interface:=hardware_interface/EffortJointInterface">
-  <xacro:property name="joint1_pos_upper_limit" value="2.90597" />    <!--  185° -->
-  <xacro:property name="joint1_pos_lower_limit" value="-2.90597" />   <!-- -185° -->
-  <xacro:property name="joint2_pos_upper_limit" value="0.942478" />   <!--   60° -->
-  <xacro:property name="joint2_pos_lower_limit" value="-2.74889" />   <!-- -175° -->
-  <xacro:property name="joint3_pos_upper_limit" value="2.67035" />    <!--  170° -->
-  <xacro:property name="joint3_pos_lower_limit" value="-1.88496" />   <!-- -120° -->
-  <xacro:property name="joint4_pos_upper_limit" value="2.82743" />    <!--  180° -->
-  <xacro:property name="joint4_pos_lower_limit" value="-2.82743" />   <!-- -180° -->
-  <xacro:property name="joint5_pos_upper_limit" value="1.9635" />     <!--  125° -->
-  <xacro:property name="joint5_pos_lower_limit" value="-1.9635" />    <!-- -125° -->
-  <xacro:property name="joint6_pos_upper_limit" value="5.49779" />    <!--  350° -->
-  <xacro:property name="joint6_pos_lower_limit" value="-5.49779" />   <!-- -350° -->
-  <xacro:property name="joint1_vel_limit" value="2.74889" />    <!--  175°/s -->
-  <xacro:property name="joint2_vel_limit" value="2.48186" />    <!--  158°/s -->
-  <xacro:property name="joint3_vel_limit" value="2.74889" />    <!--  175°/s -->
-  <xacro:property name="joint4_vel_limit" value="3.92699" />    <!--  250°/s -->
-  <xacro:property name="joint5_vel_limit" value="3.92699" />    <!--  250°/s -->
-  <xacro:property name="joint6_vel_limit" value="5.65487" />    <!--  360°/s -->
+<xacro:macro name="kr_50_r2500"  params="prefix:='' interface:=hardware_interface/EffortJointInterface">
+  <xacro:property name="joint1_pos_upper_limit" value="3.22886" />    <!--  185° -->
+  <xacro:property name="joint1_pos_lower_limit" value="-3.22886" />   <!-- -185° -->
+  <xacro:property name="joint2_pos_upper_limit" value="1.0472" />     <!--   60° -->
+  <xacro:property name="joint2_pos_lower_limit" value="-3.05433" />   <!-- -175° -->
+  <xacro:property name="joint3_pos_upper_limit" value="2.96706" />    <!--  170° -->
+  <xacro:property name="joint3_pos_lower_limit" value="-2.0944" />    <!-- -120° -->
+  <xacro:property name="joint4_pos_upper_limit" value="3.14159" />    <!--  180° -->
+  <xacro:property name="joint4_pos_lower_limit" value="-3.14159" />   <!-- -180° -->
+  <xacro:property name="joint5_pos_upper_limit" value="2.18166" />    <!--  125° -->
+  <xacro:property name="joint5_pos_lower_limit" value="-2.18166" />   <!-- -125° -->
+  <xacro:property name="joint6_pos_upper_limit" value="6.10865" />    <!--  350° -->
+  <xacro:property name="joint6_pos_lower_limit" value="-6.10865" />   <!-- -350° -->
+  <xacro:property name="joint1_vel_limit" value="3.05433" />    <!--  175°/s -->
+  <xacro:property name="joint2_vel_limit" value="2.75762" />    <!--  158°/s -->
+  <xacro:property name="joint3_vel_limit" value="3.05433" />    <!--  175°/s -->
+  <xacro:property name="joint4_vel_limit" value="4.36332" />    <!--  250°/s -->
+  <xacro:property name="joint5_vel_limit" value="4.36332" />    <!--  250°/s -->
+  <xacro:property name="joint6_vel_limit" value="6.28319" />    <!--  360°/s -->
   <xacro:property name="joint1_eff_limit" value="10000" />
   <xacro:property name="joint2_eff_limit" value="10000" />
@@ -47,5 +47,5 @@
       <geometry>
         <mesh
-          filename="package://kr_50_r2500_gazebo/meshes/base_link.STL" />
+          filename="package://kr_50_r2500_description/meshes/base_link.STL" />
       </geometry>
       <material
@@ -61,5 +61,5 @@
       <geometry>
         <mesh
-          filename="package://kr_50_r2500_gazebo/meshes/base_link.STL" />
+          filename="package://kr_50_r2500_description/meshes/base_link.STL" />
       </geometry>
     </collision>
@@ -86,19 +86,19 @@
       <geometry>
         <mesh
-          filename="package://kr_50_r2500_gazebo/meshes/link1.STL" />
-      </geometry>
-      <material
-        name="">
-        <color
-          rgba="0.792156862745098 0.819607843137255 0.933333333333333 1" />
-      </material>
-    </visual>
-    <collision>
-      <origin
-        xyz="0 0 0"
-        rpy="0 0 0" />
-      <geometry>
-        <mesh
-          filename="package://kr_50_r2500_gazebo/meshes/link1.STL" />
+          filename="package://kr_50_r2500_description/meshes/link1.STL" />
+      </geometry>
+      <material
+        name="">
+        <color
+          rgba="0.792156862745098 0.819607843137255 0.933333333333333 1" />
+      </material>
+    </visual>
+    <collision>
+      <origin
+        xyz="0 0 0"
+        rpy="0 0 0" />
+      <geometry>
+        <mesh
+          filename="package://kr_50_r2500_description/meshes/link1.STL" />
       </geometry>
     </collision>
@@ -138,19 +138,19 @@
       <geometry>
         <mesh
-          filename="package://kr_50_r2500_gazebo/meshes/link2.STL" />
-      </geometry>
-      <material
-        name="">
-        <color
-          rgba="0.792156862745098 0.819607843137255 0.933333333333333 1" />
-      </material>
-    </visual>
-    <collision>
-      <origin
-        xyz="0 0 0"
-        rpy="0 0 0" />
-      <geometry>
-        <mesh
-          filename="package://kr_50_r2500_gazebo/meshes/link2.STL" />
+          filename="package://kr_50_r2500_description/meshes/link2.STL" />
+      </geometry>
+      <material
+        name="">
+        <color
+          rgba="0.792156862745098 0.819607843137255 0.933333333333333 1" />
+      </material>
+    </visual>
+    <collision>
+      <origin
+        xyz="0 0 0"
+        rpy="0 0 0" />
+      <geometry>
+        <mesh
+          filename="package://kr_50_r2500_description/meshes/link2.STL" />
       </geometry>
     </collision>
@@ -190,19 +190,19 @@
       <geometry>
         <mesh
-          filename="package://kr_50_r2500_gazebo/meshes/link3.STL" />
-      </geometry>
-      <material
-        name="">
-        <color
-          rgba="0.792156862745098 0.819607843137255 0.933333333333333 1" />
-      </material>
-    </visual>
-    <collision>
-      <origin
-        xyz="0 0 0"
-        rpy="0 0 0" />
-      <geometry>
-        <mesh
-          filename="package://kr_50_r2500_gazebo/meshes/link3.STL" />
+          filename="package://kr_50_r2500_description/meshes/link3.STL" />
+      </geometry>
+      <material
+        name="">
+        <color
+          rgba="0.792156862745098 0.819607843137255 0.933333333333333 1" />
+      </material>
+    </visual>
+    <collision>
+      <origin
+        xyz="0 0 0"
+        rpy="0 0 0" />
+      <geometry>
+        <mesh
+          filename="package://kr_50_r2500_description/meshes/link3.STL" />
       </geometry>
     </collision>
@@ -242,19 +242,19 @@
       <geometry>
         <mesh
-          filename="package://kr_50_r2500_gazebo/meshes/link4.STL" />
-      </geometry>
-      <material
-        name="">
-        <color
-          rgba="0.792156862745098 0.819607843137255 0.933333333333333 1" />
-      </material>
-    </visual>
-    <collision>
-      <origin
-        xyz="0 0 0"
-        rpy="0 0 0" />
-      <geometry>
-        <mesh
-          filename="package://kr_50_r2500_gazebo/meshes/link4.STL" />
+          filename="package://kr_50_r2500_description/meshes/link4.STL" />
+      </geometry>
+      <material
+        name="">
+        <color
+          rgba="0.792156862745098 0.819607843137255 0.933333333333333 1" />
+      </material>
+    </visual>
+    <collision>
+      <origin
+        xyz="0 0 0"
+        rpy="0 0 0" />
+      <geometry>
+        <mesh
+          filename="package://kr_50_r2500_description/meshes/link4.STL" />
       </geometry>
     </collision>
@@ -294,19 +294,19 @@
       <geometry>
         <mesh
-          filename="package://kr_50_r2500_gazebo/meshes/link5.STL" />
-      </geometry>
-      <material
-        name="">
-        <color
-          rgba="0.792156862745098 0.819607843137255 0.933333333333333 1" />
-      </material>
-    </visual>
-    <collision>
-      <origin
-        xyz="0 0 0"
-        rpy="0 0 0" />
-      <geometry>
-        <mesh
-          filename="package://kr_50_r2500_gazebo/meshes/link5.STL" />
+          filename="package://kr_50_r2500_description/meshes/link5.STL" />
+      </geometry>
+      <material
+        name="">
+        <color
+          rgba="0.792156862745098 0.819607843137255 0.933333333333333 1" />
+      </material>
+    </visual>
+    <collision>
+      <origin
+        xyz="0 0 0"
+        rpy="0 0 0" />
+      <geometry>
+        <mesh
+          filename="package://kr_50_r2500_description/meshes/link5.STL" />
       </geometry>
     </collision>
@@ -346,19 +346,19 @@
       <geometry>
         <mesh
-          filename="package://kr_50_r2500_gazebo/meshes/link6.STL" />
-      </geometry>
-      <material
-        name="">
-        <color
-          rgba="0.792156862745098 0.819607843137255 0.933333333333333 1" />
-      </material>
-    </visual>
-    <collision>
-      <origin
-        xyz="0 0 0"
-        rpy="0 0 0" />
-      <geometry>
-        <mesh
-          filename="package://kr_50_r2500_gazebo/meshes/link6.STL" />
+          filename="package://kr_50_r2500_description/meshes/link6.STL" />
+      </geometry>
+      <material
+        name="">
+        <color
+          rgba="0.792156862745098 0.819607843137255 0.933333333333333 1" />
+      </material>
+    </visual>
+    <collision>
+      <origin
+        xyz="0 0 0"
+        rpy="0 0 0" />
+      <geometry>
+        <mesh
+          filename="package://kr_50_r2500_description/meshes/link6.STL" />
       </geometry>
     </collision>
@@ -399,6 +399,4 @@
   <xacro:include filename="$(find kr_50_r2500_description)/urdf/kr_50_r2500_transmission.xacro" />
   <xacro:kr_50_r2500_transmission prefix="${prefix}" interface="${interface}"/>
-  <xacro:include filename="$(find kr_50_r2500_description)/urdf/kr_50_r2500_gazebo.xacro" />
-  <xacro:kr_50_r2500_roscontrol prefix="${prefix}"/>
 </xacro:macro>
 </robot>

File: kr_50_r2500_description/urdf/kr_50_r2500_rviz.xacro (robot description, xacro)
@@ -3,10 +3,10 @@
   <xacro:include filename="$(find kr_50_r2500_description)/urdf/kr_50_r2500.xacro" />
   <xacro:property name="prefix" value="''" />
-<link name="world"/>
   <xacro:kr_50_r2500 prefix="${prefix}"/>
+  <link name="world"/>
   <joint name="${prefix}world_to_base_link" type="fixed">
       <origin
         xyz="0 0 0"
-        rpy="-1.57079632679 0 0" />
+        rpy="${-pi/2} 0 0" />
       <parent link="world"/>
       <child link="${prefix}base_link"/>

Commit message: some change for new simulation version

File: kr_50_r2500_description/urdf/kr_50_r2500.xacro (robot description, xacro)
@@ -26,5 +26,5 @@
   <xacro:property name="joint5_eff_limit" value="10000" />
   <xacro:property name="joint6_eff_limit" value="10000" />
-  <link name="${prefix}base_link">
+  <link name="${prefix}base_link" concave="yes">
     <inertial>
       <origin
@@ -55,5 +55,5 @@
       </material>
     </visual>
-    <collision>
+    <collision concave="yes">
       <origin
         xyz="0 0 0"
@@ -65,5 +65,5 @@
     </collision>
   </link>
-  <link name="${prefix}link1">
+  <link name="${prefix}link1" concave="yes">
     <inertial>
       <origin
@@ -94,5 +94,5 @@
       </material>
     </visual>
-    <collision>
+    <collision concave="yes">
       <origin
         xyz="0 0 0"
@@ -117,5 +117,5 @@
     <limit lower="${joint1_pos_lower_limit}" upper="${joint1_pos_upper_limit}" effort="${joint1_eff_limit}" velocity="${joint1_vel_limit}"/>
   </joint>
-  <link name="${prefix}link2">
+  <link name="${prefix}link2" concave="yes">
     <inertial>
       <origin
@@ -146,5 +146,5 @@
       </material>
     </visual>
-    <collision>
+    <collision concave="yes">
       <origin
         xyz="0 0 0"
@@ -169,5 +169,5 @@
     <limit lower="${joint2_pos_lower_limit}" upper="${joint2_pos_upper_limit}" effort="${joint2_eff_limit}" velocity="${joint2_vel_limit}"/>
   </joint>
-  <link name="${prefix}link3">
+  <link name="${prefix}link3" concave="yes">
     <inertial>
       <origin
@@ -198,5 +198,5 @@
       </material>
     </visual>
-    <collision>
+    <collision concave="yes">
       <origin
         xyz="0 0 0"
@@ -221,5 +221,5 @@
     <limit lower="${joint3_pos_lower_limit}" upper="${joint3_pos_upper_limit}" effort="${joint3_eff_limit}" velocity="${joint3_vel_limit}"/>
   </joint>
-  <link name="${prefix}link4">
+  <link name="${prefix}link4" concave="yes">
     <inertial>
       <origin
@@ -250,5 +250,5 @@
       </material>
     </visual>
-    <collision>
+    <collision concave="yes">
       <origin
         xyz="0 0 0"
@@ -273,5 +273,5 @@
     <limit lower="${joint4_pos_lower_limit}" upper="${joint4_pos_upper_limit}" effort="${joint4_eff_limit}" velocity="${joint4_vel_limit}"/>
   </joint>
-  <link name="${prefix}link5">
+  <link name="${prefix}link5" concave="yes">
     <inertial>
       <origin
@@ -302,5 +302,5 @@
       </material>
     </visual>
-    <collision>
+    <collision concave="yes">
       <origin
         xyz="0 0 0"
@@ -325,5 +325,5 @@
     <limit lower="${joint5_pos_lower_limit}" upper="${joint5_pos_upper_limit}" effort="${joint5_eff_limit}" velocity="${joint5_vel_limit}"/>
   </joint>
-  <link name="${prefix}link6">
+  <link name="${prefix}link6" concave="yes">
     <inertial>
       <origin
@@ -354,5 +354,5 @@
       </material>
     </visual>
-    <collision>
+    <collision concave="yes">
       <origin
         xyz="0 0 0"

File: kr_50_r2500_description/urdf/kr_50_r2500_pybullet.urdf (robot description, URDF)
Before this commit: robot kr_50_r2500, 8 links, 7 joints
Links:
- link base_link: geometry collision mesh filename=/home/gauss/projects/personal_ws/src/kr_50_r2500/kr_50_r250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; visual mesh filename=/home/gauss/projects/personal_ws/src/kr_50_r2500/kr_50_r250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
- link link1: geometry collision mesh filename=/home/gauss/projects/personal_ws/src/kr_50_r2500/kr_50_r250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; visual mesh filename=/home/gauss/projects/personal_ws/src/kr_50_r2500/kr_50_r250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
- link link2: geometry collision mesh filename=/home/gauss/projects/personal_ws/src/kr_50_r2500/kr_50_r250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; visual mesh filename=/home/gauss/projects/personal_ws/src/kr_50_r2500/kr_50_r250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
- link link3: geometry collision mesh filename=/home/gauss/projects/personal_ws/src/kr_50_r2500/kr_50_r250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; visual mesh filename=/home/gauss/projects/personal_ws/src/kr_50_r2500/kr_50_r250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
- link link4: geometry collision mesh filename=/home/gauss/projects/personal_ws/src/kr_50_r2500/kr_50_r250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; visual mesh filename=/home/gauss/projects/personal_ws/src/kr_50_r2500/kr_50_r250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
- link link5: geometry collision mesh filename=/home/gauss/projects/personal_ws/src/kr_50_r2500/kr_50_r250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; visual mesh filename=/home/gauss/projects/personal_ws/src/kr_50_r2500/kr_50_r250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
- link link6: geometry collision mesh filename=/home/gauss/projects/personal_ws/src/kr_50_r2500/kr_50_r250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; visual mesh filename=/home/gauss/projects/personal_ws/src/kr_50_r2500/kr_50_r250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

File: kr_50_r2500_description/urdf/kr_50_r2500_pybullet.xacro (robot description, xacro)
@@ -3,9 +3,6 @@
 <robot name="$(arg robot_name)" xmlns:xacro="http://www.ros.org/wiki/xacro">
   <xacro:include filename="$(find kr_50_r2500_description)/urdf/kr_50_r2500.xacro" />
-  <xacro:arg name="prefix" default="null"/>
+  <xacro:arg name="prefix" default=""/>
   <xacro:property name="prefix" value="'$(arg prefix)'" />
-  <xacro:if value="${prefix == 'null'}">
-    <xacro:property name="prefix" value="''" />
-  </xacro:if>
   <xacro:kr_50_r2500 prefix="${prefix}"/>
 </robot>
