Commit message: correction of numeric errors on joints origins; add new link "base" with vertical Z-axis

File: kr_50_r2500_description/urdf/kr_50_r2500_robot.xacro (robot description, xacro)
@@ -108,5 +108,5 @@
     <origin
       xyz="0 -0.17 0"
-      rpy="1.5708 0.009141 0" />
+      rpy="1.57079632679489661923 0.0 0" />
     <parent
       link="${prefix}base_link" />
@@ -160,5 +160,5 @@
     <origin
       xyz="0.175 -0.074807 0.405"
-      rpy="0 1.557055  0" />
+      rpy="0 1.57079632679489661923  0" />
     <parent
       link="${prefix}link1" />
@@ -212,5 +212,5 @@
     <origin
       xyz="0 0 1.29"
-      rpy="0 -1.557055 0" />
+      rpy="0 -1.57079632679489661923 0" />
     <parent
       link="${prefix}link2" />
@@ -316,5 +316,5 @@
     <origin
       xyz="0.708131634616243 0 0"
-      rpy="0 -0.0 0" />
+      rpy="0 0 0" />
     <parent
       link="${prefix}link4" />
@@ -380,5 +380,5 @@
       <origin
         xyz="0.07 0 0"
-        rpy="0 1.57079632679 0" />
+        rpy="0 1.57079632679489661923 0" />
       <parent link="${prefix}link6"/>
       <child link="${prefix}flange"/>

File: kr_50_r2500_description/urdf/kr_50_r2500_rviz.xacro (robot description, xacro)
@@ -11,11 +11,17 @@
                      prefix="${prefix}"
                      use_fake_hardware="${use_fake_hardware}" />
+  <link name="${prefix}base"/>
+  <joint name="${prefix}base_to_base_link" type="fixed">
+    <parent link="${prefix}base"/>
+    <child link="${prefix}base_link"/>
+    <origin rpy="-1.57079632679489661923 0 0"/>
+  </joint>
   <link name="world"/>
-  <joint name="${prefix}world_to_base_link" type="fixed">
-      <origin
+  <joint name="${prefix}world_to_base" type="fixed">
+      <!-- <origin
         xyz="0 0 0"
-        rpy="${-pi/2} 0 0" />
+        rpy="${-pi/2} 0 0" /> -->
       <parent link="world"/>
-      <child link="${prefix}base_link"/>
+      <child link="${prefix}base"/>
   </joint>
 </robot>

Commit message: initial pos

File: kr_50_r2500_description/urdf/kr_50_r2500_robot.xacro (robot description, xacro)
@@ -12,6 +12,6 @@
   <xacro:property name="joint5_pos_upper_limit" value="2.18166" />    <!--  125° -->
   <xacro:property name="joint5_pos_lower_limit" value="-2.18166" />   <!-- -125° -->
-  <xacro:property name="joint6_pos_upper_limit" value="6.10865" />    <!--  350° -->
-  <xacro:property name="joint6_pos_lower_limit" value="-6.10865" />   <!-- -350° -->
+  <xacro:property name="joint6_pos_upper_limit" value="3.14159" />    <!--  180° -->
+  <xacro:property name="joint6_pos_lower_limit" value="-4.71239" />   <!-- -270° -->
   <xacro:property name="joint1_vel_limit" value="3.05433" />    <!--  175°/s -->
   <xacro:property name="joint2_vel_limit" value="2.75762" />    <!--  158°/s -->

File: kr_50_r2500_description/urdf/kr_50_r2500_ros2_control.xacro (robot description, xacro)
@@ -37,5 +37,5 @@
         <command_interface name="position"/>
         <state_interface name="position">
-          <param name="initial_value">0.0</param>
+          <param name="initial_value">-1.5708</param>
         </state_interface>
         <state_interface name="velocity">

Commit message: Update kr_50_r2500_robot.xacro

File: kr_50_r2500_description/urdf/kr_50_r2500_robot.xacro (robot description, xacro)
@@ -26,4 +26,10 @@
   <xacro:property name="joint5_eff_limit" value="10000" />
   <xacro:property name="joint6_eff_limit" value="10000" />
+  <link name="${prefix}iksolver_base_link"/>
+  <joint name="${prefix}base_to_base_link" type="fixed">
+    <parent link="${prefix}iksolver_base_link"/>
+    <child link="${prefix}base_link"/>
+    <origin rpy="-1.57079632679489661923 0 0"/>
+  </joint>
   <link name="${prefix}base_link" concave="yes">
     <inertial>

Commit message: patch z base

File: kr_50_r2500_description/urdf/kr_50_r2500_robot.xacro (robot description, xacro)
@@ -26,15 +26,16 @@
   <xacro:property name="joint5_eff_limit" value="10000" />
   <xacro:property name="joint6_eff_limit" value="10000" />
-  <link name="${prefix}iksolver_base_link"/>
-  <joint name="${prefix}base_to_base_link" type="fixed">
-    <parent link="${prefix}iksolver_base_link"/>
-    <child link="${prefix}base_link"/>
+<!--
+  <link name="${prefix}base_link"/>
+  <joint name="${prefix}base_link_to_mesh_base" type="fixed">
+    <parent link="${prefix}base_link"/>
+    <child link="${prefix}base_link___"/>
     <origin rpy="-1.57079632679489661923 0 0"/>
-  </joint>
+  </joint>-->
   <link name="${prefix}base_link" concave="yes">
     <inertial>
       <origin
         xyz="-0.080585 0.00067592 0.086754"
-        rpy="0 0 0" />
+        rpy="-1.57079632679489661923 0 0" />
       <mass
         value="30.385" />
@@ -50,5 +51,5 @@
       <origin
         xyz="0 0 0"
-        rpy="0 0 0" />
+        rpy="-1.57079632679489661923 0 0" />
       <geometry>
         <mesh
@@ -64,5 +65,5 @@
       <origin
         xyz="0 0 0"
-        rpy="0 0 0" />
+        rpy="-1.57079632679489661923 0 0" />
       <geometry>
         <mesh
@@ -112,7 +113,5 @@
   <joint name="${prefix}joint1"
     type="revolute">
-    <origin
-      xyz="0 -0.17 0"
-      rpy="1.57079632679489661923 0.0 0" />
+    <origin      xyz="0 0 0.17"       rpy="0 0.0 0" />
     <parent
       link="${prefix}base_link" />

File: kr_50_r2500_description/urdf/kr_50_r2500_rviz.xacro (robot description, xacro)
@@ -14,5 +14,5 @@
   <joint name="${prefix}world_to_base" type="fixed">
       <parent link="world"/>
-      <child link="${prefix}iksolver_base_link"/>
+      <child link="${prefix}base_link"/>
   </joint>
 </robot>
